File: Hardware/ROBOT-CHAT_PCB/Schematic_PCB/Antenne.kicad_sch (KiCad schematic)
At the start: 5 parts

Commit message: current schematic
Parts:
- C21, C24: footprint (none) -> Capacitor_SMD:C_0402_1005Metric
- L4: footprint (none) -> Inductor_SMD:L_0603_1608Metric
- U8: footprint DLF162500LT-5028A1:LOWPASS -> LowPass:LOWPASS
Changed lines of the file:
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@@
 			)
 		)
-		(property "Footprint" ""
+		(property "Footprint" "Capacitor_SMD:C_0402_1005Metric"
 			(at 124.46 69.85 0)
 			(effects
@@
 			)
 		)
-		(property "Footprint" "DLF162500LT-5028A1:LOWPASS"
+		(property "Footprint" "LowPass:LOWPASS"
 			(at 147.32 67.31 0)
 			(effects
@@
 			)
 		)
-		(property "Footprint" ""
+		(property "Footprint" "Capacitor_SMD:C_0402_1005Metric"
 			(at 111.76 69.85 0)
 			(effects
@@
 			)
 		)
-		(property "Footprint" ""
+		(property "Footprint" "Inductor_SMD:L_0603_1608Metric"
 			(at 118.11 67.31 0)
 			(effects
