File: Hardware/ROBOT-CHAT_PCB/Schematic_PCB/PCB_robot_chat.kicad_sch (KiCad schematic)
At the start: 0 parts

Commit message: current schematic
Parts:
- added H101, H102, H103, H104: MountingHole_Pad, MountingHole:MountingHole_2.5mm_Pad_Via, symbol Mechanical:MountingHole_Pad
Connections:
- new net GND: H101.1, H102.1, H103.1, H104.1
Other:
- sheet Power ports: added none; removed EN3.3, EN5
- sheet STM ports: added none; removed EN3.3, EN5
