File: Hardware/ROBOT-CHAT_PCB/Schematic_PCB/Driver.kicad_sch (KiCad schematic)
At the start: 12 parts, among them J7 Conn_01x06, J8 Conn_01x06, U5 ZXBM5210-SP, U6 ZXBM5210-SP

Commit message: current schematic
Parts:
- J7, J8: footprint (none) -> Connector_JST:JST_PH_B6B-PH-K_1x06_P2.00mm_Vertical
Connections:
- net Moteur1+: now also U5.1 (OUT1); no longer U5.7 (OUT2)
- net Moteur1-: now also U5.7 (OUT2); no longer U5.1 (OUT1)
- net Moteur2+: now also U6.1 (OUT1); no longer U6.7 (OUT2)
- net Moteur2-: now also U6.7 (OUT2); no longer U6.1 (OUT1)
Changed lines of the file:
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@@
 	)
 	(label "Moteur2-"
-		(at 217.17 62.23 0)
+		(at 217.17 67.31 0)
 		(effects
 			(font
@@
 	)
 	(label "Moteur1+"
-		(at 92.71 64.77 0)
+		(at 92.71 59.69 0)
 		(effects
 			(font
@@
 	)
 	(label "Moteur2+"
-		(at 217.17 67.31 0)
+		(at 217.17 62.23 0)
 		(effects
 			(font
@@
 	)
 	(label "Moteur1-"
-		(at 92.71 59.69 0)
+		(at 92.71 64.77 0)
 		(effects
 			(font
@@
 			)
 		)
-		(property "Footprint" ""
+		(property "Footprint" "Connector_JST:JST_PH_B6B-PH-K_1x06_P2.00mm_Vertical"
 			(at 140.97 59.69 0)
 			(effects
@@
 			)
 		)
-		(property "Footprint" ""
+		(property "Footprint" "Connector_JST:JST_PH_B6B-PH-K_1x06_P2.00mm_Vertical"
 			(at 267.97 59.69 0)
 			(effects

Commit message: Rerouting avec Mr Fiack
Parts:
- C28, C30: footprint Capacitor_SMD:C_0603_1608Metric -> Capacitor_SMD:C_0402_1005Metric
Changed lines of the file:
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@@
 			)
 		)
-		(property "Footprint" "Capacitor_SMD:C_0603_1608Metric"
+		(property "Footprint" "Capacitor_SMD:C_0402_1005Metric"
 			(at 95.25 44.45 0)
 			(effects
@@
 			)
 		)
-		(property "Footprint" "Capacitor_SMD:C_0603_1608Metric"
+		(property "Footprint" "Capacitor_SMD:C_0402_1005Metric"
 			(at 219.71 46.99 0)
 			(effects
