File: Hardware/ROBOT-CHAT_PCB/Schematic_PCB/PCB_robot_chat.kicad_pcb (KiCad board)
At the start: 4 copper layers, 64.5 x 57 mm, 95 parts, among them J1 Conn_01x04, J201 Conn_ST_STDC14, J3 Conn_01x02, J4 Conn_01x02, J5 Conn_01x02, J501 Conn_01x04, J502 Conn_01x04, J503 Conn_01x04, J504 Conn_01x04, J6 Conn_01x02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

Commit message: Verif by Fiack, PCB version 6
Parts:
- moved C18 0.61 mm to (126.0, 51.4)
- moved C17 0.52 mm to (128.2, 49.4)
Routing:
- net Net-(U1-VLXSMPS): track 15.0 -> 11.7 mm
- net /Accéléromètre/SDAacc: track 32.9 -> 31.1 mm
- net /STM/STATUS_LEDR: track 40.4 -> 39.1 mm
- net Net-(U1-PC15): track 7.86 -> 6.67 mm, vias 2 -> 0
- net /Driver/Encodeur_2B: track 46.0 -> 44.8 mm
- net /Accéléromètre/SCLacc: track 24.9 -> 26.0 mm
- net /Accéléromètre/INTacc2: track 41.3 -> 40.3 mm
- net GND: vias 85 -> 136
